File: pcb.sch (KiCad schematic (older format))
At the start: 28 parts, among them U1 MP1580, U4 VIA, U5 VIA

Commit message: component values updated
Parts:
- C2: value 4n7 -> 10n
- C4: value 4n7 -> 220p
- C5: value 47uF -> 47uF 6.3V
- D4: value B230ADICT-ND -> B230ADICT
- L1: value 10uH -> 33uH
- R1: value 15k -> 4k7
- R2: value 10k2 1% -> 10k1%
- R3: value 34k 1% -> 33k1%
- R4: value 56 -> 150
Other:
- moved on the sheet: 12V1, 12V2, C1, D1, D2, F1, GND1, GND2
Changed lines of the file:
@@
 L Device:D_Zener D2
 U 1 1 5A8DCE57
-P 3050 3700
-F 0 "D2" H 3050 3800 50  0000 C CNN
-F 1 "TPSMA6L16A" H 3050 3600 50  0000 C CNN
-F 2 "Diodes_SMD:D_SMA" H 3050 3700 50  0001 C CNN
-F 3 "https://www.mouser.com/ds/2/240/Littelfuse_TVS_Diode_TPSMA6L_Datasheet.pdf-278015.pdf" H 3050 3700 50  0001 C CNN
-	1    3050 3700
+P 3200 3700
+F 0 "D2" H 3200 3800 50  0000 C CNN
+F 1 "TPSMA6L16A" H 3200 3600 50  0000 C CNN
+F 2 "Diodes_SMD:D_SMA" H 3200 3700 50  0001 C CNN
+F 3 "https://www.mouser.com/ds/2/240/Littelfuse_TVS_Diode_TPSMA6L_Datasheet.pdf-278015.pdf" H 3200 3700 50  0001 C CNN
+	1    3200 3700
 	0    1    1    0
 $EndComp
@@
 L Device:C C1
 U 1 1 5A8DD0BC
-P 3350 3700
-F 0 "C1" H 3375 3800 50  0000 L CNN
-F 1 "10uF/35V" H 3375 3600 50  0000 L CNN
-F 2 "Capacitors_SMD:C_1206" H 3388 3550 50  0001 C CNN
-F 3 "https://www.mouser.com/ds/2/281/c02e-2905.pdf" H 3350 3700 50  0001 C CNN
-	1    3350 3700
+P 3500 3700
+F 0 "C1" H 3525 3800 50  0000 L CNN
+F 1 "10uF/35V" H 3525 3600 50  0000 L CNN
+F 2 "Capacitors_SMD:C_1206" H 3538 3550 50  0001 C CNN
+F 3 "" H 3500 3700 50  0001 C CNN
+	1    3500 3700
 	1    0    0    -1
 $EndComp
@@
 L power:GNDD #PWR01
 U 1 1 5A8FD3FB
-P 3050 4550
-F 0 "#PWR01" H 3050 4300 50  0001 C CNN
-F 1 "GNDD" H 3050 4425 50  0001 C CNN
-F 2 "" H 3050 4550 50  0001 C CNN
-F 3 "" H 3050 4550 50  0001 C CNN
-	1    3050 4550
+P 3200 4550
+F 0 "#PWR01" H 3200 4300 50  0001 C CNN
+F 1 "GNDD" H 3200 4425 50  0001 C CNN
+F 2 "" H 3200 4550 50  0001 C CNN
+F 3 "" H 3200 4550 50  0001 C CNN
+	1    3200 4550
 	1    0    0    -1
 $EndComp
@@
 L power:GNDD #PWR02
 U 1 1 5A8FD47B
-P 3350 4550
-F 0 "#PWR02" H 3350 4300 50  0001 C CNN
-F 1 "GNDD" H 3350 4425 50  0001 C CNN
-F 2 "" H 3350 4550 50  0001 C CNN
-F 3 "" H 3350 4550 50  0001 C CNN
-	1    3350 4550
+P 3500 4550
+F 0 "#PWR02" H 3500 4300 50  0001 C CNN
+F 1 "GNDD" H 3500 4425 50  0001 C CNN
+F 2 "" H 3500 4550 50  0001 C CNN
+F 3 "" H 3500 4550 50  0001 C CNN
+	1    3500 4550
 	1    0    0    -1
 $EndComp
@@
 L Device:D D1
 U 1 1 5A8DCFD6
-P 2850 2850
-F 0 "D1" H 2850 2950 50  0000 C CNN
-F 1 "S3JB" H 2850 2750 50  0000 C CNN
-F 2 "Diodes_SMD:D_SMB" H 2850 2850 50  0001 C CNN
-F 3 "https://www.mouser.com/ds/2/395/S3AB%20SERIES_L1705-1113162.pdf" H 2850 2850 50  0001 C CNN
-	1    2850 2850
+P 3000 2850
+F 0 "D1" H 3000 2950 50  0000 C CNN
+F 1 "S3JB" H 3000 2750 50  0000 C CNN
+F 2 "Diodes_SMD:D_SMB" H 3000 2850 50  0001 C CNN
+F 3 "https://www.mouser.com/ds/2/395/S3AB%20SERIES_L1705-1113162.pdf" H 3000 2850 50  0001 C CNN
+	1    3000 2850
 	-1   0    0    1
 $EndComp
@@
 P 5100 3400
 F 0 "D4" H 5100 3500 50  0000 C CNN
-F 1 "B230ADICT-ND" H 5200 3250 50  0000 C CNN
+F 1 "B230ADICT" H 5150 3300 50  0000 C CNN
 F 2 "Diodes_SMD:D_SMB" H 5100 3400 50  0001 C CNN
 F 3 "https://www.mouser.com/ds/2/115/ds13004-70120.pdf" H 5100 3400 50  0001 C CNN
@@
 P 5400 3200
 F 0 "L1" V 5350 3200 50  0000 C CNN
-F 1 "10uH" V 5510 3200 50  0000 C CNN
+F 1 "33uH" V 5510 3200 50  0000 C CNN
 F 2 "MyKiCAD:L_Taiyo-Yuden_NR10050" H 5400 3200 50  0001 C CNN
 F 3 "https://www.mouser.com/datasheet/2/396/wound06_e-1313806.pdf" H 5400 3200 50  0001 C CNN
@@
 L power:GNDD #PWR010
 U 1 1 5A953F25
-P 2300 4550
-F 0 "#PWR010" H 2300 4300 50  0001 C CNN
-F 1 "GNDD" H 2300 4425 50  0001 C CNN
-F 2 "" H 2300 4550 50  0001 C CNN
-F 3 "" H 2300 4550 50  0001 C CNN
-	1    2300 4550
-	1    0    0    -1
-$EndComp
-Connection ~ 3350 2850
-Connection ~ 3050 2850
-Wire Wire Line
-	3050 4550 3050 3850
-Wire Wire Line
-	3000 2850 3050 2850
-Wire Wire Line
-	3050 2850 3050 3550
-Wire Wire Line
-	2300 4550 2300 4500
-Wire Wire Line
-	2300 4500 2150 4500
+P 2450 4550
+F 0 "#PWR010" H 2450 4300 50  0001 C CNN
+F 1 "GNDD" H 2450 4425 50  0001 C CNN
+F 2 "" H 2450 4550 50  0001 C CNN
+F 3 "" H 2450 4550 50  0001 C CNN
+	1    2450 4550
+	1    0    0    -1
+$EndComp
+Connection ~ 3500 2850
+Connection ~ 3200 2850
+Wire Wire Line
+	3200 4550 3200 3850
+Wire Wire Line
+	3150 2850 3200 2850
+Wire Wire Line
+	3200 2850 3200 3550
+Wire Wire Line
+	2450 4550 2450 4500
+Wire Wire Line
+	2450 4500 2300 4500
 $Comp
 L via:VIA 12V1
 U 1 1 5A954668
-P 2150 2850
-F 0 "12V1" V 2150 3050 50  0000 C CNN
-F 1 "TEST_1P" H 2150 3050 50  0001 C CNN
-F 2 "MyKiCAD:VIA-1.2-2.5MM" H 2350 2850 50  0001 C CNN
-F 3 "" H 2350 2850 50  0001 C CNN
-	1    2150 2850
+P 2300 2850
+F 0 "12V1" V 2300 3050 50  0000 C CNN
+F 1 "TEST_1P" H 2300 3050 50  0001 C CNN
+F 2 "MyKiCAD:VIA-1.2-2.5MM" H 2500 2850 50  0001 C CNN
+F 3 "" H 2500 2850 50  0001 C CNN
+	1    2300 2850
 	0    -1   -1   0
 $EndComp
@@
 L via:VIA GND2
 U 1 1 5A954755
-P 2150 4500
-F 0 "GND2" V 2150 4800 50  0000 C CNN
-F 1 "TEST_1P" H 2150 4700 50  0001 C CNN
-F 2 "MyKiCAD:VIA-1.2-2.5MM" H 2350 4500 50  0001 C CNN
-F 3 "" H 2350 4500 50  0001 C CNN
-	1    2150 4500
+P 2300 4500
+F 0 "GND2" V 2300 4800 50  0000 C CNN
+F 1 "TEST_1P" H 2300 4700 50  0001 C CNN
+F 2 "MyKiCAD:VIA-1.2-2.5MM" H 2500 4500 50  0001 C CNN
+F 3 "" H 2500 4500 50  0001 C CNN
+	1    2300 4500
 	0    -1   -1   0
 $EndComp
@@
 $EndComp
 Wire Wire Line
-	3050 2850 3350 2850
-Wire Wire Line
-	3350 2850 3350 3550
+	3200 2850 3500 2850
+Wire Wire Line
+	3500 2850 3500 3550
 $Comp
 L EnergyHarvester:MP1580 U1
@@
 	4100 2850 4100 2900
 Wire Wire Line
-	3350 2850 4100 2850
+	3500 2850 4100 2850
 $Comp
 L Device:C C3
@@
 F 1 "10n" H 4450 2750 50  0000 L CNN
 F 2 "Capacitors_SMD:C_0603" H 4638 2700 50  0001 C CNN
-F 3 "https://www.mouser.com/ds/2/281/c02e-2905.pdf" H 4600 2850 50  0001 C CNN
+F 3 "" H 4600 2850 50  0001 C CNN
 	1    4600 2850
 	0    1    1    0
@@
 P 6000 3500
 F 0 "R4" V 6080 3500 50  0000 C CNN
-F 1 "56" V 6000 3500 50  0000 C CNN
+F 1 "150" V 6000 3500 50  0000 C CNN
 F 2 "Resistors_SMD:R_0603" V 5930 3500 50  0001 C CNN
 F 3 "" H 6000 3500 50  0001 C CNN
@@
 U 1 1 5BE55A89
 P 5550 3850
-F 0 "R3" V 5630 3850 50  0000 C CNN
-F 1 "34k 1%" V 5550 3850 50  0000 C CNN
+F 0 "R3" V 5450 3850 50  0000 C CNN
+F 1 "33k1%" V 5550 3850 39  0000 C CNN
 F 2 "Resistors_SMD:R_0603" V 5480 3850 50  0001 C CNN
 F 3 "" H 5550 3850 50  0001 C CNN
@@
 P 5100 4250
 F 0 "R2" V 5180 4250 50  0000 C CNN
-F 1 "10k2 1%" V 5100 4250 50  0000 C CNN
+F 1 "10k1%" V 5100 4250 39  0000 C CNN
 F 2 "Resistors_SMD:R_0603" V 5030 4250 50  0001 C CNN
 F 3 "" H 5100 4250 50  0001 C CNN
@@
 P 5700 3400
 F 0 "C5" H 5725 3500 50  0000 L CNN
-F 1 "47uF" H 5725 3300 50  0000 L CNN
+F 1 "47uF 6.3V" H 5500 3300 50  0000 L CNN
 F 2 "Capacitors_SMD:C_0805" H 5738 3250 50  0001 C CNN
-F 3 "https://www.mouser.com/ds/2/281/c02e-2905.pdf" H 5700 3400 50  0001 C CNN
+F 3 "" H 5700 3400 50  0001 C CNN
 	1    5700 3400
 	-1   0    0    1
@@
 	5700 3200 6000 3200
 Wire Wire Line
-	2150 3000 2300 3000
-Wire Wire Line
-	2300 3000 2300 2850
-Wire Wire Line
-	2300 2850 2150 2850
+	2300 3000 2450 3000
+Wire Wire Line
+	2450 3000 2450 2850
+Wire Wire Line
+	2450 2850 2300 2850
 $Comp
 L via:VIA 12V2
 U 1 1 5BE88EFD
-P 2150 3000
-F 0 "12V2" V 2150 3200 50  0000 C CNN
-F 1 "TEST_1P" H 2150 3200 50  0001 C CNN
-F 2 "MyKiCAD:VIA-1.2-2.5MM" H 2350 3000 50  0001 C CNN
-F 3 "" H 2350 3000 50  0001 C CNN
-	1    2150 3000
+P 2300 3000
+F 0 "12V2" V 2300 3200 50  0000 C CNN
+F 1 "TEST_1P" H 2300 3200 50  0001 C CNN
+F 2 "MyKiCAD:VIA-1.2-2.5MM" H 2500 3000 50  0001 C CNN
+F 3 "" H 2500 3000 50  0001 C CNN
+	1    2300 3000
 	0    -1   -1   0
 $EndComp
@@
 L via:VIA GND1
 U 1 1 5BE88F45
-P 2150 4350
-F 0 "GND1" V 2150 4650 50  0000 C CNN
-F 1 "TEST_1P" H 2150 4550 50  0001 C CNN
-F 2 "MyKiCAD:VIA-1.2-2.5MM" H 2350 4350 50  0001 C CNN
-F 3 "" H 2350 4350 50  0001 C CNN
-	1    2150 4350
+P 2300 4350
+F 0 "GND1" V 2300 4650 50  0000 C CNN
+F 1 "TEST_1P" H 2300 4550 50  0001 C CNN
+F 2 "MyKiCAD:VIA-1.2-2.5MM" H 2500 4350 50  0001 C CNN
+F 3 "" H 2500 4350 50  0001 C CNN
+	1    2300 4350
 	0    -1   -1   0
 $EndComp
 Wire Wire Line
-	2150 4350 2300 4350
-Wire Wire Line
-	2300 4350 2300 4500
-Connection ~ 2300 4500
+	2300 4350 2450 4350
+Wire Wire Line
+	2450 4350 2450 4500
+Connection ~ 2450 4500
 $Comp
 L Device:R R1
@@
 P 4400 4350
 F 0 "R1" V 4480 4350 50  0000 C CNN
-F 1 "15k" V 4400 4350 50  0000 C CNN
+F 1 "4k7" V 4400 4350 50  0000 C CNN
 F 2 "Resistors_SMD:R_0603" V 4330 4350 50  0001 C CNN
 F 3 "" H 4400 4350 50  0001 C CNN
@@
 P 4400 4000
 F 0 "C2" H 4425 4100 50  0000 L CNN
-F 1 "4n7" H 4425 3900 50  0000 L CNN
+F 1 "10n" H 4425 3900 50  0000 L CNN
 F 2 "Capacitors_SMD:C_0603" H 4438 3850 50  0001 C CNN
-F 3 "https://www.mouser.com/ds/2/281/c02e-2905.pdf" H 4400 4000 50  0001 C CNN
+F 3 "" H 4400 4000 50  0001 C CNN
 	1    4400 4000
 	-1   0    0    1
@@
 U 1 1 5BE8A7B8
 P 4700 4150
-F 0 "C4" H 4725 4250 50  0000 L CNN
-F 1 "4n7" H 4725 4050 50  0000 L CNN
+F 0 "C4" H 4550 4250 50  0000 L CNN
+F 1 "220p" H 4500 4050 50  0000 L CNN
 F 2 "Capacitors_SMD:C_0603" H 4738 4000 50  0001 C CNN
-F 3 "https://www.mouser.com/ds/2/281/c02e-2905.pdf" H 4700 4150 50  0001 C CNN
+F 3 "" H 4700 4150 50  0001 C CNN
 	1    4700 4150
 	-1   0    0    1
@@
 	6200 4000 6200 3650
 Wire Wire Line
-	3350 3850 3350 4550
+	3500 3850 3500 4550
 $Comp
 L Device:Fuse F1
 U 1 1 5BF1FC9C
-P 2500 2850
-F 0 "F1" V 2303 2850 50  0000 C CNN
-F 1 "5A Fast Blow" V 2394 2850 50  0000 C CNN
-F 2 "MyKiCAD:LittleFuse Fast Fuse Axial" V 2430 2850 50  0001 C CNN
-F 3 "https://www.mouser.com/datasheet/2/240/Littelfuse_Fuse_251_253_Datasheet.pdf-522535.pdf" H 2500 2850 50  0001 C CNN
-	1    2500 2850
-	0    1    1    0
-$EndComp
-Wire Wire Line
-	2700 2850 2650 2850
-Wire Wire Line
-	2300 2850 2350 2850
-Connection ~ 2300 2850
+P 2650 2850
+F 0 "F1" V 2750 2850 50  0000 C CNN
+F 1 "5A Fast Blow" V 2550 2800 50  0000 C CNN
+F 2 "MyKiCAD:LittleFuse Fast Fuse Axial" V 2580 2850 50  0001 C CNN
+F 3 "https://www.mouser.com/datasheet/2/240/Littelfuse_Fuse_251_253_Datasheet.pdf-522535.pdf" H 2650 2850 50  0001 C CNN
+	1    2650 2850
+	0    1    1    0
+$EndComp
+Wire Wire Line
+	2850 2850 2800 2850
+Wire Wire Line
+	2450 2850 2500 2850
+Connection ~ 2450 2850
 $EndSCHEMATC
